File: PCB/ele713/ele713.kicad_sch (KiCad schematic)
At the start: 64 parts, among them Q1 PMBT2222A-Q, Q2 PMBT2907A-Q, T1 Vi = 36-72V, Vo = 12V / 1.25A, U1 LM5012, U2 LT8304, U3 UCC28C55, U4 ISOM8110, U5 TL431DBZ

Commit message: libraries added, schematic fully completed except terminals
Parts:
- added C28, C29: 22u, Capacitor_THT:CP_Radial_D10.0mm_P5.00mm, symbol Device:C_Polarized_Small_US
- added C30, C31: 3.3u, powerlabLibrary:R46KN410050N1K, symbol Device:C
- added C32, C33, C34, C35: 4.7u, Capacitor_SMD:C_1210_3225Metric_Pad1.33x2.70mm_HandSolder, symbol Device:C
- added C36, C37, C38, C39: 22u, Capacitor_SMD:C_1210_3225Metric_Pad1.33x2.70mm_HandSolder, symbol Device:C
- added C40, C41: 2.2u, powerlabLibrary:F861KM473M310A, symbol Device:C
- added C42, C43: 220u, powerlabLibrary:CAPAE830X1250N, symbol Device:C_Polarized_Small_US
- added D4: V35PWL63, Package_TO_SOT_SMD:TO-252-2, symbol powerlabLibrary:V35PWL63
- added D5, D6: SDT5H100LP5, powerlabLibrary:D_PowerDI-5, symbol powerlabLibrary:SDT5H100LP5
- added D7, D8: BZT52H-A18-QX, Diode_SMD:D_SOD-123F, symbol powerlabLibrary:BZT52H-A18-QX
- added J1, J2: Conn_01x02_Pin, TerminalBlock_RND:TerminalBlock_RND_205-00067_1x02_P7.50mm_Horizontal, symbol Connector:Conn_01x02_Pin
- added PS1: SC-18-10J, powerlabLibrary:SC1810J, symbol powerlabLibrary:SC-18-10J
- added Q3, Q4: BSC096N10LS5, Package_TO_SOT_SMD:TDSON-8-1, symbol powerlabLibrary:BSC096N10LS5
- added R24, R25: 10R, Diode_SMD:D_1206_3216Metric_Pad1.42x1.75mm_HandSolder, symbol Device:R_US
- added R26, R27: 100k, Resistor_SMD:R_0805_2012Metric_Pad1.20x1.40mm_HandSolder, symbol Device:R_US
- added T2: ELE713 Transformer, powerlabLibrary:ETD39_coilformer, symbol Device:Transformer_1P_1S
- added U6: 2EDB8259F, Package_SO:SOIC-16_3.9x9.9mm_P1.27mm, symbol powerlabLibrary:2EDB8259F
- C19: footprint Capacitor_THT:C_Rect_L10.0mm_W3.0mm_P7.50mm_MKS4 -> powerlabLibrary:R76QD0220SE00J
- D1: footprint Diode_SMD:D_PowerDI-5 -> powerlabLibrary:D_PowerDI-5
- U3: footprint Package_SO:VSSOP-8_3x3mm_P0.65mm -> powerlabLibrary:VSSOP-8_3x3mm_P0.65mm
- U4: footprint Package_SO:SOIC-4_4.55x3.7mm_P2.54mm -> powerlabLibrary:SOIC-4_4.55x3.7mm_P2.54mm
Connections:
- net +12V: now also U6.11 (VDDB), U6.3 (VDDI), U6.8 (VDDI)
- net GND: now also C28.2, C29.2, C30.2, C31.2, C32.2, C33.2, C34.2, C35.2, D6.2 (A), PS1.3 (N2_1), U6.4 (GNDI), U6.5 (DIS), U6.6 (STP/DTC), U6.9 (GNDB)
- net ISO12: now also U6.16 (VDDA)
- net ISOGND: now also D6.1 (K), D7.2 (A), Q4.1 (S), Q4.2 (S), Q4.3 (S), R27.2, T2.1 (AA), U6.14 (GNDA)
- net OUTGND: now also C36.2, C37.2, C38.2, C39.2, C40.2, C41.2, C42.2, C43.2, J2.2 (Pin_2), T2.3 (SA)
- net VIN: now also C28.1, C29.1, C30.1, C31.1, C32.1, C33.1, C34.1, C35.1, D5.1 (K), PS1.4 (N2_2), Q4.5 (D)
- net Vo: now also C36.1, C37.1, C38.1, C39.1, C40.1, C41.1, C42.1, C43.1, D4.2 (K), J2.1 (Pin_1)
- net LS_SOURCE: now reaches R10.1, R14.1
- net LS_SOURCE: now also D8.2 (A), Q3.1 (S), Q3.2 (S), Q3.3 (S), R26.2
- net GATE renamed PWM
- net PWM: now also U6.1 (INA), U6.2 (INB)
- new net: D5.2 (A), Q3.5 (D), T2.2 (AB)
- new net: D4.1 (A), D4.3 (A), T2.4 (SB)
- new net: D7.1 (K), Q4.4 (G), R24.2, R27.1
- new net: J1.2 (Pin_2), PS1.1 (N1_1)
- new net: J1.1 (Pin_1), PS1.2 (N1_2)
- new net: D8.1 (K), Q3.4 (G), R25.2, R26.1
- new net GATE_HIGH: R24.1, U6.15 (OUTA)
- new net GATE_LOW: R25.1, U6.10 (OUTB)
Other:
- note added: "36-72V to 12V Buck"
- note added: "36-72V to Isolated 12V Flyback"
- note added: "Input Filter"
- note added: "Output Filter"
- note added: "Two-Switch Flyback Controller"
- note added: "Two-Switch Flyback Converter"
- note added: "Two-channel Gate Driver"
- moved on the sheet: C1, C10, C11, C12, C13, C14, C15, C16, C17, C18, C19, C2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
