File: PCB/ele713_ozdisan/ele713_ozdisan/ele713_ozdisan.kicad_sch (KiCad schematic)
At the start: 80 parts, among them J1 Conn_01x02_Pin, J2 Conn_01x02_Pin, Q1 FDD86110, Q2 FDD86110, Q5 PZT2222AT1G, Q6 PZT2907AT1G, T2 ELE713 Transformer, U1 2EDS8265H, U2 LM5576MHX_NOPB, U3 TCMT1103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

Commit message: PCB v1 ve v2 çizildi
Çok sancılı bir süreç, ilk PCB yi çizmek zormuş yıprandım. Neyse, v1 ve v2 çizildi. V2 basılacak olan şimdilik.
Parts:
- added F1: Fuse, Fuse:Fuseholder_Cylinder-5x20mm_Schurter_0031_8201_Horizontal_Open, symbol Device:Fuse
- added J3, J4: Conn_01x10, Connector_PinHeader_2.54mm:PinHeader_1x10_P2.54mm_Vertical, symbol Connector_Generic:Conn_01x10
Connections:
- net +12V: now also J4.9 (Pin_9)
- net GND: now also C15.2, U1.4 (GNDI), U1.5 (DISABLE), U1.8 (SLDON), J3.10 (Pin_10), J4.7 (Pin_7), J4.8 (Pin_8)
- net ISO12: now also C17.2; no longer C17.1
- net ISOGND: now also C17.1; no longer C17.2
- net VIN: now also F1.2, J3.3 (Pin_3), J3.4 (Pin_4); no longer J1.1 (Pin_1)
- net LM5576_11: now reaches C1.1, U2.11 (SS)
- net LM5576_11: now also J4.10 (Pin_10)
- net LM5576_8: now reaches R4.1, U2.8 (RT)
- net LM5576_8: now also J3.8 (Pin_8)
- net LM5576_7: now reaches R2.2, R3.1, U2.7 (FB)
- net LM5576_7: now also J3.7 (Pin_7)
- net LM5576_6: now reaches C3.1, R1.1, U2.6 (COMP)
- net LM5576_6: now also J3.6 (Pin_6)
- net LM5576_20: now reaches C6.1, U2.20 (BST)
- net LM5576_20: now also J4.1 (Pin_1)
- net LM5576_17: now reaches C6.2, D2.2 (K), L1.1, U2.17 (SW_2), U2.18 (SW), U2.19 (PRE)
- net LM5576_17: now also J4.2 (Pin_2), J4.3 (Pin_3), J4.4 (Pin_4)
- net LM5576_1: now reaches C2.1, U2.1 (VCC)
- net LM5576_1: now also J3.1 (Pin_1)
- net LM5576_9: now reaches C4.1, U2.9 (RAMP)
- net LM5576_9: now also J3.9 (Pin_9)
- net LM5576_15: now reaches D2.1 (A), D2.3 (A), U2.15 (IS_2), U2.16 (IS)
- net LM5576_15: now also J4.5 (Pin_5), J4.6 (Pin_6)
- net LM5576_2: now reaches U2.2 (SD)
- net LM5576_2: now also J3.2 (Pin_2)
- net LM5576_5: now reaches U2.5 (SYNC)
- net LM5576_5: now also J3.5 (Pin_5)
- new net VIN_UNPROTECTED: F1.1, J1.1 (Pin_1)
Other:
- moved on the sheet: C17, J1
